File: pcb/mainboard/M.2 E&M Key.kicad_sch (KiCad schematic)
At the start: 26 parts, among them J15 Bus_M.2_Socket_M, J16 Bus_M.2_Socket_E

Commit message: before i start jul 10th
Parts:
- removed H7, H8: MountingHole_M2.0, A_HDJ_Library:MountingHole_2.7mm_M2_Pad_TopOnly, symbol Mechanical:MountingHole_Pad
